File: no-escape.kicad_pcb (KiCad board)
At the start: 2 copper layers, 246.6 x 75.1 mm, 116 parts, among them J1 SM04B, J2 SWD, SW1 Boot, U1 RP2040, U2 XC6206PxxxMR, U3 W25Q128JVS, U4 PRTR5V0U2X, Y1 12MHz

Commit message: add 1.5 1 bottom compatibility
Parts:
- added MX45: win, parts:mx_1u, F.Cu at (61.9, 101.6)
- added MX46: ctrl, parts:mx_15u, F.Cu at (38.1, 101.6)
- MX44: value 8U -> space
- moved D37 7.33 mm to (70.0, 102.5)
- moved D36 7.21 mm to (46.0, 102.5)
Routing:
- net ROW4: track 212.6 -> 205.4 mm
- net Net-(D37-A): track 4.55 -> 11.6 mm
- net Net-(D36-A): track 4.55 -> 11.4 mm
- net GND: vias 11 -> 12
